File: kicad/state mode logic analyzer.kicad_pcb (KiCad board)
At the start: 4 copper layers, 82.8 x 56.7 mm, 134 parts, among them J1 USB0, J2 Exp Out, J5 Exp In, J6 Probe, J7 SWD0, J8 Probe Power, J9 5V USB0, SW1 Reset 0, SW2 Boot 0, U1 RP2040, U10 74LVC245APW, U11 74LVC245APW, U3 74HC4520D, U4 LTC6994xS6-1, U5 MCP4725, U6 AD5241BRZ1M, U7 IS25LP128F-JBLE, U9 MCP1826S, Y1 ECS-120-18-33-JEM-TR

Commit message: gerbers plotted for fab
Parts:
- moved H3 0.48 mm to (180.0, 102.3)
- moved H1 0.47 mm to (193.8, 70.1)
Changed lines of the file:
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@@
     )
     (pad_to_mask_clearance 0)
-    (solder_mask_min_width 0.1016)
+    (allow_soldermask_bridges_in_footprints yes)
     (pcbplotparams
       (layerselection 0x00010fc_ffffffff)
@@
       (plotinvisibletext false)
       (sketchpadsonfab false)
-      (subtractmaskfromsilk false)
+      (subtractmaskfromsilk true)
       (outputformat 1)
       (mirror false)
-      (drillshape 1)
+      (drillshape 0)
       (scaleselection 1)
       (outputdirectory "")
@@
   )
   (footprint "MountingHole:MountingHole_2.7mm" (layer "F.Cu")
-    (at 194.025 69.7)
+    (at 193.75 70.075)
     (descr "Mounting Hole 2.7mm, no annular")
     (tags "mounting hole 2.7mm no annular")
@@
     (fp_line (start 1.6 0.8) (end 1.6 -0.8)
       (stroke (width 0.1) (type solid)) (layer "F.Fab"))
-    (pad "1" smd roundrect (at -1.4875 0 90) (size 1.425 1.75) (layers "F.Cu" "F.Paste" "F.Mask") (roundrect_rratio 0.175439)
+    (pad "1" smd roundrect (at -1.4875 0 90) (size 1.425 1.75) (layers "F.Cu" "F.Paste" "F.Mask") (roundrect_rratio 0.1754392982)
       (net 1 "GND") (pinfunction "K") (pintype "passive"))
-    (pad "2" smd roundrect (at 1.4875 0 90) (size 1.425 1.75) (layers "F.Cu" "F.Paste" "F.Mask") (roundrect_rratio 0.175439)
+    (pad "2" smd roundrect (at 1.4875 0 90) (size 1.425 1.75) (layers "F.Cu" "F.Paste" "F.Mask") (roundrect_rratio 0.1754392982)
       (net 8 "Net-(D3-A)") (pinfunction "A") (pintype "passive"))
     (model "${KICAD6_3DMODEL_DIR}/LED_SMD.3dshapes/LED_1206_3216Metric.wrl"
@@
     (fp_line (start 1.6 0.8) (end 1.6 -0.8)
       (stroke (width 0.1) (type solid)) (layer "F.Fab"))
-    (pad "1" smd roundrect (at -1.4875 0 90) (size 1.425 1.75) (layers "F.Cu" "F.Paste" "F.Mask") (roundrect_rratio 0.175439)
+    (pad "1" smd roundrect (at -1.4875 0 90) (size 1.425 1.75) (layers "F.Cu" "F.Paste" "F.Mask") (roundrect_rratio 0.1754392982)
       (net 1 "GND") (pinfunction "K") (pintype "passive"))
-    (pad "2" smd roundrect (at 1.4875 0 90) (size 1.425 1.75) (layers "F.Cu" "F.Paste" "F.Mask") (roundrect_rratio 0.175439)
+    (pad "2" smd roundrect (at 1.4875 0 90) (size 1.425 1.75) (layers "F.Cu" "F.Paste" "F.Mask") (roundrect_rratio 0.1754392982)
       (net 10 "Net-(D5-A)") (pinfunction "A") (pintype "passive"))
     (model "${KICAD6_3DMODEL_DIR}/LED_SMD.3dshapes/LED_1206_3216Metric.wrl"
@@
     (fp_line (start 1.6 0.8) (end 1.6 -0.8)
       (stroke (width 0.1) (type solid)) (layer "F.Fab"))
-    (pad "1" smd roundrect (at -1.4875 0 90) (size 1.425 1.75) (layers "F.Cu" "F.Paste" "F.Mask") (roundrect_rratio 0.175439)
+    (pad "1" smd roundrect (at -1.4875 0 90) (size 1.425 1.75) (layers "F.Cu" "F.Paste" "F.Mask") (roundrect_rratio 0.1754392982)
       (net 1 "GND") (pinfunction "K") (pintype "passive"))
-    (pad "2" smd roundrect (at 1.4875 0 90) (size 1.425 1.75) (layers "F.Cu" "F.Paste" "F.Mask") (roundrect_rratio 0.175439)
+    (pad "2" smd roundrect (at 1.4875 0 90) (size 1.425 1.75) (layers "F.Cu" "F.Paste" "F.Mask") (roundrect_rratio 0.1754392982)
       (net 9 "Net-(D4-A)") (pinfunction "A") (pintype "passive"))
     (model "${KICAD6_3DMODEL_DIR}/LED_SMD.3dshapes/LED_1206_3216Metric.wrl"
@@
     (fp_line (start 1.6 0.8) (end 1.6 -0.8)
       (stroke (width 0.1) (type solid)) (layer "F.Fab"))
-    (pad "1" smd roundrect (at -1.4875 0 90) (size 1.425 1.75) (layers "F.Cu" "F.Paste" "F.Mask") (roundrect_rratio 0.175439)
+    (pad "1" smd roundrect (at -1.4875 0 90) (size 1.425 1.75) (layers "F.Cu" "F.Paste" "F.Mask") (roundrect_rratio 0.1754392982)
       (net 1 "GND") (pinfunction "K") (pintype "passive"))
-    (pad "2" smd roundrect (at 1.4875 0 90) (size 1.425 1.75) (layers "F.Cu" "F.Paste" "F.Mask") (roundrect_rratio 0.175439)
+    (pad "2" smd roundrect (at 1.4875 0 90) (size 1.425 1.75) (layers "F.Cu" "F.Paste" "F.Mask") (roundrect_rratio 0.1754392982)
       (net 6 "Net-(D1-A)") (pinfunction "A") (pintype "passive"))
     (model "${KICAD6_3DMODEL_DIR}/LED_SMD.3dshapes/LED_1206_3216Metric.wrl"
@@
     (fp_line (start 1.6 0.8) (end 1.6 -0.8)
       (stroke (width 0.1) (type solid)) (layer "F.Fab"))
-    (pad "1" smd roundrect (at -1.4875 0 90) (size 1.425 1.75) (layers "F.Cu" "F.Paste" "F.Mask") (roundrect_rratio 0.175439)
+    (pad "1" smd roundrect (at -1.4875 0 90) (size 1.425 1.75) (layers "F.Cu" "F.Paste" "F.Mask") (roundrect_rratio 0.1754392982)
       (net 1 "GND") (pinfunction "K") (pintype "passive"))
-    (pad "2" smd roundrect (at 1.4875 0 90) (size 1.425 1.75) (layers "F.Cu" "F.Paste" "F.Mask") (roundrect_rratio 0.175439)
+    (pad "2" smd roundrect (at 1.4875 0 90) (size 1.425 1.75) (layers "F.Cu" "F.Paste" "F.Mask") (roundrect_rratio 0.1754392982)
       (net 11 "Net-(D6-A)") (pinfunction "A") (pintype "passive"))
     (model "${KICAD6_3DMODEL_DIR}/LED_SMD.3dshapes/LED_1206_3216Metric.wrl"
@@
   )
   (footprint "MountingHole:MountingHole_2.7mm" (layer "F.Cu")
-    (at 179.5 102.375)
+    (at 179.975 102.35)
     (descr "Mounting Hole 2.7mm, no annular")
     (tags "mounting hole 2.7mm no annular")
@@
     (fp_line (start 3.5 3.5) (end -3.5 3.5)
       (stroke (width 0.1) (type solid)) (layer "F.Fab"))
-    (pad "" smd roundrect (at -0.8 -0.8 45) (size 1.29 1.29) (layers "F.Paste") (roundrect_rratio 0.193798))
-    (pad "" smd roundrect (at -0.8 0.8 45) (size 1.29 1.29) (layers "F.Paste") (roundrect_rratio 0.193798))
-    (pad "" smd roundrect (at 0.8 -0.8 45) (size 1.29 1.29) (layers "F.Paste") (roundrect_rratio 0.193798))
-    (pad "" smd roundrect (at 0.8 0.8 45) (size 1.29 1.29) (layers "F.Paste") (roundrect_rratio 0.193798))
+    (pad "" smd roundrect (at -0.8 -0.8 45) (size 1.29 1.29) (layers "F.Paste") (roundrect_rratio 0.1937976744))
+    (pad "" smd roundrect (at -0.8 0.8 45) (size 1.29 1.29) (layers "F.Paste") (roundrect_rratio 0.1937976744))
+    (pad "" smd roundrect (at 0.8 -0.8 45) (size 1.29 1.29) (layers "F.Paste") (roundrect_rratio 0.1937976744))
+    (pad "" smd roundrect (at 0.8 0.8 45) (size 1.29 1.29) (layers "F.Paste") (roundrect_rratio 0.1937976744))
     (pad "1" smd roundrect (at -3.4375 -2.6 45) (size 0.875 0.2) (layers "F.Cu" "F.Paste" "F.Mask") (roundrect_rratio 0.25)
       (net 4 "+3V3") (pinfunction "IOVDD") (pintype "power_in"))
@@
     (fp_line (start 1.6 0.8) (end 1.6 -0.8)
       (stroke (width 0.1) (type solid)) (layer "F.Fab"))
-    (pad "1" smd roundrect (at -1.4875 0 90) (size 1.425 1.75) (layers "F.Cu" "F.Paste" "F.Mask") (roundrect_rratio 0.175439)
+    (pad "1" smd roundrect (at -1.4875 0 90) (size 1.425 1.75) (layers "F.Cu" "F.Paste" "F.Mask") (roundrect_rratio 0.1754392982)
       (net 1 "GND") (pinfunction "K") (pintype "passive"))
-    (pad "2" smd roundrect (at 1.4875 0 90) (size 1.425 1.75) (layers "F.Cu" "F.Paste" "F.Mask") (roundrect_rratio 0.175439)
+    (pad "2" smd roundrect (at 1.4875 0 90) (size 1.425 1.75) (layers "F.Cu" "F.Paste" "F.Mask") (roundrect_rratio 0.1754392982)
       (net 7 "Net-(D2-A)") (pinfunction "A") (pintype "passive"))
     (model "${KICAD6_3DMODEL_DIR}/LED_SMD.3dshapes/LED_1206_3216Metric.wrl"
@@
   (gr_rect (start 177.29375 71.034374) (end 182.875 75)
     (stroke (width 0.254) (type default)) (fill none) (layer "F.SilkS"))
-  (gr_rect (start -4.425 -2.775) (end 0 0)
-    (stroke (width 0.254) (type default)) (fill none) (layer "F.SilkS"))
   (gr_circle (center 134.25 106.225) (end 134.15 106.325)
     (stroke (width 0.15) (type default)) (fill none) (layer "F.SilkS"))
@@
   (gr_rect (start 119.1 82.5375) (end 121.875 86.9625)
     (stroke (width 0.254) (type default)) (fill none) (layer "F.SilkS"))
-  (gr_rect (start 156.325 77.5625) (end 156.775 78.8375)
-    (stroke (width 0.1) (type solid)) (fill solid) (layer "F.Mask"))
-  (gr_rect (start 163.2 81.45) (end 164.475 81.9)
-    (stroke (width 0.1) (type solid)) (fill solid) (layer "F.Mask"))
-  (gr_rect (start 156.3 74.85) (end 156.75 76.125)
-    (stroke (width 0.1) (type solid)) (fill solid) (layer "F.Mask"))
-  (gr_rect (start 159.0125 81.45) (end 160.2875 81.9)
-    (stroke (width 0.1) (type solid)) (fill solid) (layer "F.Mask"))
-  (gr_rect (start 164.175 87.8) (end 165.45 88.25)
-    (stroke (width 0.1) (type solid)) (fill solid) (layer "F.Mask"))
   (gr_rect (start 118.55 66.3) (end 201.325 123)
     (stroke (width 0.1) (type default)) (fill none) (layer "Edge.Cuts"))
