File: kicad/state mode logic analyzer.kicad_pcb (KiCad board)
At the start: 4 copper layers, 82.8 x 56.7 mm, 134 parts, among them J1 USB0, J2 Exp Out, J5 Exp In, J6 Probe, J7 SWD0, J8 Probe Power, J9 5V USB0, SW1 Reset 0, SW2 Boot 0, U1 RP2040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

Commit message: fixed J desgs and swapped prog header part num
Parts:
- moved C2 65.8 mm to (92.8, 69.2)
- moved C31 65.8 mm to (74.8, 67.8)
- moved C8 65.8 mm to (85.4, 62.0)
- moved C10 65.8 mm to (84.8, 55.1)
- moved C11 65.8 mm to (81.1, 55.5)
- moved C19 65.8 mm to (103.8, 50.0)
- moved C20 65.8 mm to (111.8, 41.4)
- moved C23 65.8 mm to (138.8, 77.0)
- moved C24 65.8 mm to (138.8, 82.1)
- moved C7 65.8 mm to (88.5, 54.5)
- moved C9 65.8 mm to (79.1, 60.0)
- moved H1 65.8 mm to (138.8, 34.0)
- moved H2 65.8 mm to (71.5, 43.0)
- moved J1 65.8 mm to (67.3, 58.1)
- moved J6 65.8 mm to (143.0, 82.1)
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- renumbered J9 to J2, J2 to J3, J5 to J4, J6 to J5, J8 to J6
